Commit message: Add training log, configuration, and model files for PPO agent. Implemented YAML configuration for training parameters, enhanced logging, and created necessary directories for model artifacts. Updated environment and URDF files for improved control and stability.

File: worm_rl/urdf/worm.urdf (robot description, URDF)
Before this commit: robot worm, 6 links, 5 joints
Links:
- link worm_link_0: mass 0.2 -> 0.1
- link worm_link_1: mass 0.2 -> 0.1
- link worm_link_2: mass 0.2 -> 0.1
- link worm_link_3: mass 0.2 -> 0.1
- link worm_link_4: mass 0.2 -> 0.1
- link worm_link_5: mass 0.2 -> 0.1
Joints:
- joint worm_joint_0: limit lower=-0.5 upper=0.5 effort=2.0 velocity=1.0 -> lower=-1.0 upper=1.0 effort=5.0 velocity=3.0
- joint worm_joint_1: limit lower=-0.5 upper=0.5 effort=2.0 velocity=1.0 -> lower=-1.0 upper=1.0 effort=5.0 velocity=3.0
- joint worm_joint_2: limit lower=-0.5 upper=0.5 effort=2.0 velocity=1.0 -> lower=-1.0 upper=1.0 effort=5.0 velocity=3.0
- joint worm_joint_3: limit lower=-0.5 upper=0.5 effort=2.0 velocity=1.0 -> lower=-1.0 upper=1.0 effort=5.0 velocity=3.0
- joint worm_joint_4: limit lower=-0.5 upper=0.5 effort=2.0 velocity=1.0 -> lower=-1.0 upper=1.0 effort=5.0 velocity=3.0
